File: src/pcbs/form-zero/form-zero.kicad_pcb (KiCad board)
At the start: 2 copper layers, 228.6 x 95.2 mm, 124 parts, among them J1 Conn_01x17_Pin, SW1 SW_Push, SW10 SW_Push, SW11 SW_Push, SW12 SW_Push, SW13 SW_Push, SW14 SW_Push, SW15 SW_Push, SW16 SW_Push, SW17 SW_Push, SW18 SW_Push, SW19 SW_Push, SW2 SW_Push, SW20 SW_Push, SW21 SW_Push, SW22 SW_Push, SW23 SW_Push, SW24 SW_Push, SW25 SW_Push, SW26 SW_Push, SW27 SW_Push, SW28 SW_Push, SW29 SW_Push, SW3 SW_Push, SW30 SW_Push, SW31 SW_Push, SW32 SW_Push, SW33 SW_Push, SW34 SW_Push, SW35 SW_Push, SW36 SW_Push, SW37 SW_Push, SW38 SW_Push, SW39 SW_Push, SW4 SW_Push, SW40 SW_Push, SW41 SW_Push, SW42 SW_Push, SW43 SW_Push, SW44 SW_Push, SW45 SW_Push, SW46 SW_Push, SW47 SW_Push, SW48 SW_Push, SW49 SW_Push, SW5 SW_Push, SW50 SW_Push, SW51 SW_Push, SW52 SW_Push, SW53 SW_Push, SW54 SW_Push, SW55 SW_Push, SW56 SW_Push, SW57 SW_Push, SW58 SW_Push, SW59 SW_Push, SW6 SW_Push, SW60 SW_Push, SW61 SW_Push, SW7 SW_Push, SW8 SW_Push, SW9 SW_Push

Commit message: add bottom row: 1.25, 1.25, 7, 1.25, 1.25
Parts:
- added S7: MX_stab, PCM_marbastlib-mx:STAB_MX_7u, F.Cu at (135.6, 108.7)
- added SW62: SW_Push, PCM_marbastlib-mx:SW_MX_HS_CPG151101S11_1.25u, B.Cu at (33.2, 108.7)
- added SW63: SW_Push, PCM_marbastlib-mx:SW_MX_HS_CPG151101S11_1.25u, B.Cu at (57.0, 108.7)
- added SW64: SW_Push, PCM_marbastlib-mx:SW_MX_HS_CPG151101S11_1.25u, B.Cu at (214.2, 108.7)
- added SW65: SW_Push, PCM_marbastlib-mx:SW_MX_HS_CPG151101S11_1.25u, B.Cu at (238.0, 108.7)
- moved D50 12.2 mm to (50.5, 99.1), turned to 180 degrees
- moved D49 12.2 mm to (31.4, 99.1), turned to 180 degrees
- moved D57 11.2 mm to (204.7, 99.1), turned to 0 degrees
- moved D58 11.2 mm to (223.7, 99.1), turned to 0 degrees
- moved D59 11.2 mm to (242.8, 99.1), turned to 0 degrees
Routing:
- net Net-(D58-A): track 3.03 -> 18.1 mm
- net col1: track 152.3 -> 166.6 mm
- net Net-(D50-A): track 3.03 -> 15.7 mm
- net Net-(D49-A): track 3.03 -> 15.2 mm
- net row4: track 254.9 -> 266.3 mm
- net Net-(D59-A): track 3.03 -> 13.6 mm
- net col10: track 144.7 -> 155.1 mm
- net col0: track 175.4 -> 184.5 mm
- net col11: track 167.8 -> 176.0 mm
- net Net-(D57-A): track 3.03 -> 5.34 mm
